File: AirQ.kicad_sch (KiCad schematic)
At the start: 0 parts

Commit message: Add: Project Files
Other:
- company: (none) -> Julian Sanchez
- title: (none) -> AirQ
Changed lines of the file:
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@@
 	(generator_version "9.0")
 	(paper "A4")
+	(title_block
+		(title "AirQ")
+		(date "2026-06-25")
+		(rev "1")
+		(company "Julian Sanchez")
+	)
 	(sheet_instances
 		(path "/"
