File: AirQ.kicad_sch (KiCad schematic)
At the start: 18 parts, among them P1 USB_C_Plug_USB2.0, SW1 EN, U1 ESP32-H2-MINI-1-H2, U2 AP2112K-3.3, U3 AP2112K-1.8

Commit message: changes
Parts:
- added U4: ENS210, Package_DFN_QFN:AMS_QFN-4-1EP_2x2mm_P0.95mm_EP0.7x1.6mm, symbol Sensor_Humidity:ENS210
- added U5: ENS161-BLGM, ENS161-BLGM:XDCR_ENS161-BLGM, symbol ENS161-BLGM:ENS161-BLGM
Connections:
- net GND: now also U4.4 (GND), U4.5 (GND), U5.8 (VSS)
- new net VSS: U5.9 (VSS)

Commit message: Avances Viernes
Parts:
- removed C4: 1uF, symbol Device:C
- removed R2: 5.1K, symbol Device:R_US
- removed R5: 10K, symbol Device:R_US
- removed U3: AP2112K-1.8, Package_TO_SOT_SMD:SOT-23-5, symbol Regulator_Linear:AP2112K-1.8
- added C1, C5, C7, C8: 1uF, Capacitor_SMD:C_0201_0603Metric, symbol Device:C
- added C10, C11, C12, C14: 0.1uF, Capacitor_SMD:C_0402_1005Metric, symbol Device:C
- added C13: 10uF, Capacitor_SMD:C_0402_1005Metric, symbol Device:C
- added D3, D4, D5: WS2812B, LED_SMD:LED_WS2812B_PLCC4_5.0x5.0mm_P3.2mm, symbol LED:WS2812B
- added Q1: BSS138, Package_TO_SOT_SMD:SOT-23, symbol Transistor_FET:BSS138
- added R1, R6, R7, R8: 10K, Resistor_SMD:R_0402_1005Metric, symbol Device:R_US
- added R10, R11, R12, R13: 4.7K, Resistor_SMD:R_0805_2012Metric, symbol Device:R_US
- added R3: 5.1K, Resistor_SMD:R_1206_3216Metric_Pad1.30x1.75mm_HandSolder, symbol Device:R_US
- added R9: 470, Resistor_SMD:R_1206_3216Metric, symbol Device:R_US
- added SW2: EN, Button_Switch_SMD:SW_Push_1P1T_NO_CK_KMR2, symbol Switch:SW_Push
- C2: value 1uF -> 10uF; footprint (none) -> Capacitor_SMD:C_0402_1005Metric; DigiKey Part Number (none) -> 490-GRM155R60J106ME05DCT-ND; Manufacturer (none) -> Murata Electronics; Manufacturer Product Number (none) -> GRM155R60J106ME05D
- C3: value 1uF -> 0.1uF; footprint (none) -> Capacitor_SMD:C_0402_1005Metric; DigiKey Part Number (none) -> 1276-1002-6-ND; Manufacturer (none) -> Samsung Electro-Mechanics; Manufacturer Product Number (none) -> CL05B104KP5NNNC
- C4: renamed from C1; footprint (none) -> Capacitor_SMD:C_0201_0603Metric; DigiKey Part Number (none) -> 541-0.0JTR-ND; Manufacturer (none) -> Vishay Dale; Manufacturer Product Number (none) -> CRCW04020000Z0ED
- C6: footprint (none) -> Capacitor_SMD:C_0201_0603Metric; DigiKey Part Number (none) -> 541-0.0JTR-ND; Manufacturer (none) -> Vishay Dale; Manufacturer Product Number (none) -> CRCW04020000Z0ED
- C9: renamed from C5; footprint (none) -> Capacitor_SMD:C_0402_1005Metric; DigiKey Part Number (none) -> 1276-1002-6-ND; Manufacturer (none) -> Samsung Electro-Mechanics; Manufacturer Product Number (none) -> CL05B104KP5NNNC
- D1: DigiKey Part Number (none) -> 1801-SS12TR-ND; Manufacturer (none) -> Taiwan Semiconductor Corporation; Manufacturer Product Number (none) -> SS12
- D2: footprint (none) -> LED_SMD:LED_0603_1608Metric; DigiKey Part Number (none) -> SML-D12U1WT86CT-ND; Manufacturer (none) -> Rohm Semiconductor; Manufacturer Product Number (none) -> SML-D12U1WT86
- P1: footprint (none) -> Connector_USB:USB_C_Receptacle_GCT_USB4105-xx-A_16P_TopMnt_Horizontal; DigiKey Part Number (none) -> 2223-UJ20-C-H-G-SMT-1-P16-TR-ND; Manufacturer (none) -> Same Sky (Formerly CUI Devices); Manufacturer Product Number (none) -> UJ20-C-H-G-SMT-1-P16-TR
- R2: renamed from R1; footprint (none) -> Resistor_SMD:R_1206_3216Metric_Pad1.30x1.75mm_HandSolder; DigiKey Part Number (none) -> 541-D55342K07B5H10RS2CT-ND; Manufacturer (none) -> Vishay Dale; Manufacturer Product Number (none) -> D55342K07B5H10RS2
- R4: value 5.1K -> 10K; footprint (none) -> Resistor_SMD:R_0402_1005Metric; DigiKey Part Number (none) -> 541-M55342K11B10E0RS3CT-ND; Manufacturer (none) -> Vishay Dale; Manufacturer Product Number (none) -> M55342K11B10E0RS3
- R5: renamed from R3; footprint (none) -> Resistor_SMD:R_0805_2012Metric; DigiKey Part Number (none) -> 541-M55342K06B330GRS2CT-ND; Manufacturer (none) -> Vishay Dale; Manufacturer Product Number (none) -> M55342K06B330GRS2
- SW1: footprint (none) -> Button_Switch_SMD:SW_Push_1P1T_NO_CK_KMR2
- U1: Availability In Stock -> (none); Check_prices https://www.snapeda.com/parts/ESP32-H2-MINI-1-H2/Espressif+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 -> (none); Description_1 802.15.4, Bluetooth Bluetooth v5.3, Zigbee® Transceiver Mod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 -> (none); DigiKey Part Number (none) -> 1965-ESP32-H2-MINI-1-H2SCT-ND; MANUFACTURER Espressif Systems -> (none); MAXIMUM_PACKAGE_HEIGHT 2.55mm -> (none); MF Espressif Systems -> (none); MP ESP32-H2-MINI-1-H2 -> (none); Manufacturer (none) -> Espressif Systems; Manufacturer Product Number (none) -> ESP32-H2-MINI-1-H2S; PARTREV v0.5 -> (none); Package SMD-53 Espressif Systems -> (none); Price None -> (none); SNAPEDA_PN ESP32-H2-MINI-1-H2 -> (none); STANDARD Manufacturer Recommendations -> (none); SnapEDA_Link https://www.snapeda.com/parts/ESP32-H2-MINI-1-H2/Espressif+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 -> (none)
- U2: DigiKey Part Number (none) -> AP2112K-3.3TRG1DICT-ND; Manufacturer (none) -> Diodes Incorporated; Manufacturer Product Number (none) -> AP2112K-3.3TRG1
- U3: renamed from U4; DigiKey Part Number (none) -> 2618-ENS210-LQFMCT-ND; Manufacturer (none) -> ScioSense; Manufacturer Product Number (none) -> ENS210-LQFM
- U4: renamed from U5; footprint ENS161-BLGM:XDCR_ENS161-BLGM -> ENS161:XDCR_ENS161-BLGM; Availability In Stock -> (none); Check_prices https://www.snapeda.com/parts/ENS161-BLGM/ScioSense/view-pa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 -> (none); Description_1 Versatile digital air quality sensor for building automatio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 -> (none); DigiKey Part Number (none) -> 2618-ENS161-BLGTCT-ND; MANUFACTURER Sciosense -> (none); MAXIMUM_PACKAGE_HEIGHT 0.9 mm -> (none); MF ScioSense -> (none); MP ENS161-BLGM -> (none); Manufacturer (none) -> ScioSense; Manufacturer Product Number (none) -> ENS161-BLGT; PARTREV 1.3 -> (none); Package LGA-9 ScioSense -> (none); Price None -> (none); STANDARD Manufacturer Recommendations -> (none); SnapEDA_Link https://www.snapeda.com/parts/ENS161-BLGM/ScioSense/view-pa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 -> (none)
Connections:
- net VSS is gone; now on net GND: U4.9 (VSS)
- net +3.3V: now also U3.1 (VDD), U4.4 (VDD), U4.5 (VDDIO), U4.7 (~{CS}), C13.1, C14.1, C5.1, C7.1, Q1.1 (G), R1.2, R10.1, R11.1, R12.1, R13.1, R6.2, R7.2
- net +5V: now also C10.1, C11.1, C12.1, D3.1 (VDD), D4.1 (VDD), D5.1 (VDD), R8.2
- net D+: now also U1.27 (IO27), C8.1; no longer U1.25 (IO25)
- net D-: now also C6.1
- net GND: now also U4.3 (MISO/ADDR), C1.2, C10.2, C11.2, C12.2, C13.2, C14.2, C5.2, C7.2, C8.2, D3.3 (VSS), D4.3 (VSS), D5.3 (VSS), R3.2, SW2.1
- net RESET: now also C1.1, R1.1, R7.1; no longer C6.1, R4.2
- net SCL: now reaches U3.2 (SCL)
- net SCL: now also U1.10 (IO01), U4.1 (MOSI/SDA), R10.2, R13.2
- net SDA: now reaches U3.3 (SDA)
- net SDA: now also U1.9 (IO0), U4.2 (SCLK/SCL), R11.2, R12.2
- net at P1.A5 (CC): now also R3.1
- net at U1.22 (IO08): now also R4.2
- net BOOT: now reaches U1.23 (IO9)
- net BOOT: now also SW2.2
- net LED_P: now reaches U1.24 (IO22)
- net LED_P: now also Q1.2 (S), R6.1
- net at U1.4 (NC): no longer U1.5 (IO2)
- new net: D4.2 (DOUT), D5.4 (DIN)
- new net: D3.2 (DOUT), D4.4 (DIN)
- new net: D3.4 (DIN), R9.1
- new net: Q1.3 (D), R8.1, R9.2
- no-connect marks 9 -> 24
Other:
- moved on the sheet: C9, SW1, U1, U3, U4
